Commit message: [modify]depth coordinate gap

File: zed_wrapper/urdf/zed.urdf.xacro (robot description, xacro)
@@ -69,5 +69,31 @@
             </inertial>
         </link>
-    <!-- Left Camera -->
+        <!-- camera depth joints and links -->
+        <joint name="$(arg camera_name)_depth_joint" type="fixed">
+            <origin xyz="0 0 0" rpy="0 0 0"/>
+            <parent link="$(arg camera_name)_camera_center"/>
+            <child link="$(arg camera_name)_depth_frame" />
+        </joint>
+        <link name="$(arg camera_name)_depth_frame"/>
+        <joint name="$(arg camera_name)_depth_optical_joint" type="fixed">
+            <origin xyz="0 0 0" rpy="-${M_PI/2} 0.0 -${M_PI/2}" />
+            <parent link="$(arg camera_name)_depth_frame" />
+            <child link="$(arg camera_name)_depth_optical_frame" />
+        </joint>
+        <link name="$(arg camera_name)_depth_optical_frame"/>
+        <!-- camera color joints and links -->
+        <joint name="$(arg camera_name)_color_joint" type="fixed">
+            <origin xyz="0 0 0" rpy="0 0 0"/>
+            <parent link="$(arg camera_name)_camera_center"/>
+            <child link="$(arg camera_name)_color_frame" />
+        </joint>
+        <link name="$(arg camera_name)_color_frame"/>
+        <joint name="$(arg camera_name)_color_optical_joint" type="fixed">
+            <origin xyz="0 0 0" rpy="-${M_PI/2} 0.0 -${M_PI/2}" />
+            <parent link="$(arg camera_name)_color_frame" />
+            <child link="$(arg camera_name)_color_optical_frame" />
+        </joint>
+        <link name="$(arg camera_name)_color_optical_frame"/>
+        <!-- Left Camera -->
         <joint name="$(arg camera_name)_left_camera_joint" type="fixed">
             <parent link="$(arg camera_name)_camera_center"/>
@@ -82,5 +108,5 @@
         </joint>
         <link name="$(arg camera_name)_left_camera_optical_frame"/>
-    <!-- Right Camera -->
+        <!-- Right Camera -->
         <joint name="$(arg camera_name)_right_camera_joint" type="fixed">
             <parent link="$(arg camera_name)_camera_center"/>
@@ -94,6 +120,6 @@
             <child link="$(arg camera_name)_right_camera_optical_frame"/>
         </joint>
-        <link name="$(arg camera_name)_right_camera_optical_frame"/>
-    <!-- ZED2 Sensors -->
+    <link name="$(arg camera_name)_right_camera_optical_frame"/>
+        <!-- ZED2 Sensors -->
         <xacro:if value="${model == 'zed2'}">
             <joint name="$(arg camera_name)_mag_joint" type="fixed">
@@ -122,5 +148,5 @@
             <link name="$(arg camera_name)_temp_right_link" />
         </xacro:if>
-        <xacro:gazebo_zed camera_name="$(arg camera_name)" reference_link="$(arg camera_name)_camera_center" topics_ns="${topics_ns}" depth_optical_frame="$(arg camera_name)_depth_optical_frame" color_optical_frame="$(arg camera_name)_color_optical_frame" infrared1_optical_frame="$(arg camera_name)_left_ir_optical_frame" infrared2_optical_frame="$(arg camera_name)_right_ir_optical_frame"/>
+        <xacro:gazebo_zed camera_name="$(arg camera_name)" reference_link="$(arg camera_name)_camera_center" topics_ns="topics_ns" depth_optical_frame="$(arg camera_name)_depth_optical_frame" color_optical_frame="$(arg camera_name)_color_optical_frame" />
     </xacro:macro>
 </robot>

File: zed_wrapper/urdf/zed_descr.urdf.xacro (robot description, xacro)
@@ -70,4 +70,30 @@
         </inertial>
     </link>
+        <!-- camera depth joints and links -->
+        <joint name="$(arg camera_name)_depth_joint" type="fixed">
+            <origin xyz="0 0 0" rpy="0 0 0"/>
+            <parent link="$(arg camera_name)_camera_center"/>
+            <child link="$(arg camera_name)_depth_frame" />
+        </joint>
+        <link name="$(arg camera_name)_depth_frame"/>
+        <joint name="$(arg camera_name)_depth_optical_joint" type="fixed">
+        <origin xyz="0 0 0" rpy="-${M_PI/2} 0.0 -${M_PI/2}" />
+        <parent link="$(arg camera_name)_depth_frame" />
+        <child link="$(arg camera_name)_depth_optical_frame" />
+        </joint>
+        <link name="$(arg camera_name)_depth_optical_frame"/>
+        <!-- camera color joints and links -->
+        <joint name="$(arg camera_name)_color_joint" type="fixed">
+            <origin xyz="0 0 0" rpy="0 0 0"/>
+            <parent link="$(arg camera_name)_camera_center"/>
+            <child link="$(arg camera_name)_color_frame" />
+            </joint>
+            <link name="$(arg camera_name)_color_frame"/>
+            <joint name="$(arg camera_name)_color_optical_joint" type="fixed">
+            <origin xyz="0 0 0" rpy="-${M_PI/2} 0.0 -${M_PI/2}" />
+            <parent link="$(arg camera_name)_color_frame" />
+            <child link="$(arg camera_name)_color_optical_frame" />
+            </joint>
+            <link name="$(arg camera_name)_color_optical_frame"/>
 <!-- Left Camera -->
     <joint name="$(arg camera_name)_left_camera_joint" type="fixed">
@@ -123,4 +149,4 @@
         <link name="$(arg camera_name)_temp_right_link" />
     </xacro:if>
-    <xacro:gazebo_zed camera_name="$(arg camera_name)" reference_link="$(arg camera_name)_camera_center" topics_ns="topics_ns" depth_optical_frame="$(arg camera_name)_depth_optical_frame" color_optical_frame="$(arg camera_name)_color_optical_frame" infrared1_optical_frame="$(arg camera_name)_left_ir_optical_frame" infrared2_optical_frame="$(arg camera_name)_right_ir_optical_frame"/>
+    <xacro:gazebo_zed camera_name="$(arg camera_name)" reference_link="$(arg camera_name)_camera_center" topics_ns="topics_ns" depth_optical_frame="$(arg camera_name)_depth_optical_frame" color_optical_frame="$(arg camera_name)_color_optical_frame" />
 </robot>

File: zed_wrapper/urdf/zed_gazebo.xacro (robot description, xacro)
@@ -8,5 +8,5 @@
     <xacro:arg name="camera_name"   default="zed" />
     <xacro:arg name="base_frame"    default="base_link" />
-    <xacro:macro name="gazebo_zed" params="camera_name reference_link topics_ns depth_optical_frame color_optical_frame infrared1_optical_frame infrared2_optical_frame" >
+    <xacro:macro name="gazebo_zed" params="camera_name reference_link topics_ns depth_optical_frame color_optical_frame " >
         <!-- Load parameters to model's main link-->
         <xacro:property name="deg_to_rad" value="0.01745329251994329577" />
@@ -51,5 +51,5 @@
                 <imageTopicName>/color/image_raw</imageTopicName>
                 <cameraInfoTopicName>/color/camera_info</cameraInfoTopicName>
-                <frameName>$(arg camera_name)_left_camera_optical_frame</frameName>
+                <frameName>${color_optical_frame}</frameName>
                 <hackBaseline>0.07</hackBaseline>
                 <distortionK1>0.0</distortionK1>
@@ -91,5 +91,5 @@
                 <depthImageCameraInfoTopicName>/${camera_name}/depth/camera_info</depthImageCameraInfoTopicName>
                 <pointCloudTopicName>/${camera_name}/depth/points</pointCloudTopicName>
-                <frameName>$(arg camera_name)_left_camera_optical_frame</frameName>
+                <frameName>${depth_optical_frame}</frameName>
                 <pointCloudCutoff>0.3</pointCloudCutoff>
                 <pointCloudCutoffMax>25.0</pointCloudCutoffMax>
