Commit message: [add]zed gazebo model

File: zed_wrapper/urdf/zed_descr.urdf.xacro (robot description, xacro)
@@ -18,4 +18,5 @@
 <!-- Includes -->
     <xacro:include filename="$(find zed_wrapper)/urdf/include/materials.urdf.xacro" />
+    <xacro:include filename="$(find zed_wrapper)/urdf/zed_gazebo.xacro"/>
     <!-- Arguments -->
     <xacro:arg name="camera_name"   default="zed" />
@@ -56,4 +57,16 @@
             <material name="${model}_mat" />
         </visual>
+        <collision>
+            <origin xyz="0 0.0175 0" rpy="0 0 0"/>
+            <geometry>
+            <box size="0.02505 0.090 0.025"/>
+            </geometry>
+        </collision>
+        <inertial>
+            <!-- The following are not reliable values, and should not be used for modeling -->
+            <mass value="0.564" />
+            <origin xyz="0 0 0" />
+            <inertia ixx="0.003881243" ixy="0.0" ixz="0.0" iyy="0.000498940" iyz="0.0" izz="0.003879257" />
+        </inertial>
     </link>
 <!-- Left Camera -->
@@ -110,3 +123,4 @@
         <link name="$(arg camera_name)_temp_right_link" />
     </xacro:if>
+    <xacro:gazebo_zed camera_name="$(arg camera_name)" reference_link="$(arg camera_name)_camera_center" topics_ns="topics_ns" depth_optical_frame="$(arg camera_name)_depth_optical_frame" color_optical_frame="$(arg camera_name)_color_optical_frame" infrared1_optical_frame="$(arg camera_name)_left_ir_optical_frame" infrared2_optical_frame="$(arg camera_name)_right_ir_optical_frame"/>
 </robot>

Commit message: [Add]zed model no macro

File: zed_wrapper/urdf/zed_descr.urdf.xacro (robot description, xacro)
@@ -70,31 +70,31 @@
         </inertial>
     </link>
-        <!-- camera depth joints and links -->
-        <joint name="$(arg camera_name)_depth_joint" type="fixed">
-            <origin xyz="0 0 0" rpy="0 0 0"/>
-            <parent link="$(arg camera_name)_camera_center"/>
-            <child link="$(arg camera_name)_depth_frame" />
-        </joint>
-        <link name="$(arg camera_name)_depth_frame"/>
-        <joint name="$(arg camera_name)_depth_optical_joint" type="fixed">
+    <!-- camera depth joints and links -->
+    <joint name="$(arg camera_name)_depth_joint" type="fixed">
+        <origin xyz="0 0 0" rpy="0 0 0"/>
+        <parent link="$(arg camera_name)_camera_center"/>
+        <child link="$(arg camera_name)_depth_frame" />
+    </joint>
+    <link name="$(arg camera_name)_depth_frame"/>
+    <joint name="$(arg camera_name)_depth_optical_joint" type="fixed">
         <origin xyz="0 0 0" rpy="-${M_PI/2} 0.0 -${M_PI/2}" />
         <parent link="$(arg camera_name)_depth_frame" />
         <child link="$(arg camera_name)_depth_optical_frame" />
-        </joint>
-        <link name="$(arg camera_name)_depth_optical_frame"/>
-        <!-- camera color joints and links -->
-        <joint name="$(arg camera_name)_color_joint" type="fixed">
-            <origin xyz="0 0 0" rpy="0 0 0"/>
-            <parent link="$(arg camera_name)_camera_center"/>
-            <child link="$(arg camera_name)_color_frame" />
-            </joint>
-            <link name="$(arg camera_name)_color_frame"/>
-            <joint name="$(arg camera_name)_color_optical_joint" type="fixed">
-            <origin xyz="0 0 0" rpy="-${M_PI/2} 0.0 -${M_PI/2}" />
-            <parent link="$(arg camera_name)_color_frame" />
-            <child link="$(arg camera_name)_color_optical_frame" />
-            </joint>
-            <link name="$(arg camera_name)_color_optical_frame"/>
-<!-- Left Camera -->
+    </joint>
+    <link name="$(arg camera_name)_depth_optical_frame"/>
+    <!-- camera color joints and links -->
+    <joint name="$(arg camera_name)_color_joint" type="fixed">
+        <origin xyz="0 0 0" rpy="0 0 0"/>
+        <parent link="$(arg camera_name)_camera_center"/>
+        <child link="$(arg camera_name)_color_frame" />
+    </joint>
+    <link name="$(arg camera_name)_color_frame"/>
+    <joint name="$(arg camera_name)_color_optical_joint" type="fixed">
+        <origin xyz="0 0 0" rpy="-${M_PI/2} 0.0 -${M_PI/2}" />
+        <parent link="$(arg camera_name)_color_frame" />
+        <child link="$(arg camera_name)_color_optical_frame" />
+    </joint>
+    <link name="$(arg camera_name)_color_optical_frame"/>
+    <!-- Left Camera -->
     <joint name="$(arg camera_name)_left_camera_joint" type="fixed">
         <parent link="$(arg camera_name)_camera_center"/>
@@ -109,5 +109,5 @@
     </joint>
     <link name="$(arg camera_name)_left_camera_optical_frame"/>
-<!-- Right Camera -->
+    <!-- Right Camera -->
     <joint name="$(arg camera_name)_right_camera_joint" type="fixed">
         <parent link="$(arg camera_name)_camera_center"/>
@@ -121,6 +121,6 @@
         <child link="$(arg camera_name)_right_camera_optical_frame"/>
     </joint>
-    <link name="$(arg camera_name)_right_camera_optical_frame"/>
-<!-- ZED2 Sensors -->
+<link name="$(arg camera_name)_right_camera_optical_frame"/>
+    <!-- ZED2 Sensors -->
     <xacro:if value="${model == 'zed2'}">
         <joint name="$(arg camera_name)_mag_joint" type="fixed">
